Commit message: modify tf

File: limo_ros2/limo_description/urdf/limo_four_diff.xacro (robot description, xacro)
@@ -72,6 +72,6 @@
         <origin xyz="${-wheelbase/2} ${-track/2} ${wheel_vertical_offset}" rpy="${M_PI} 0 0" />
     </xacro:limo_wheel>
-    <gazebo reference="imu_link">
-    <gravity>true</gravity>
+    <!-- <gazebo reference="imu_link"> -->
+    <!-- <gravity>true</gravity>
     <sensor name="twr_imu" type="imu">
       <always_on>true</always_on>
@@ -149,6 +149,6 @@
       </plugin>
     </sensor>
-</gazebo>
-<gazebo reference="laser_link">
+</gazebo> -->
+<!-- <gazebo reference="laser_link">
     <sensor name="laser" type="ray">
       <always_on>true</always_on>
@@ -183,6 +183,6 @@
       </plugin>
     </sensor>
-  </gazebo>
-    <gazebo reference="front_left_wheel">
+  </gazebo> -->
+    <!-- <gazebo reference="front_left_wheel">
         <mu1>100</mu1>
         <mu2>100</mu2>
@@ -244,5 +244,5 @@
         </ros>
         </plugin>
-    </gazebo>
+    </gazebo> -->
         <!-- <gazebo reference="depth_camera_link">
           <sensor name="sensor_camera" type="depth">

File: limo_ros2/limo_description/urdf/limo_xacro.xacro (robot description, xacro)
@@ -68,5 +68,5 @@
         </gazebo>
     </xacro:macro>
-    <xacro:macro name="limo_depth_camera" params="parent_prefix frame_prefix *joint_pose">
+    <!-- <xacro:macro name="limo_depth_camera" params="parent_prefix frame_prefix *joint_pose">
         <link name='${frame_prefix}_link'>
             <pose>0 0 0 0 0 0</pose>
@@ -79,5 +79,5 @@
                     izz="1e-6"
                 />
-            </inertial>
+            </inertial> -->
             <!-- <visual name='depth_camera_visual'>
                 <origin xyz="0 0 0" rpy="0 0 0"/>
@@ -92,5 +92,5 @@
                 </material>
             </visual> -->
-            <collision name='depth_camera_collision'>
+            <!-- <collision name='depth_camera_collision'>
                 <origin xyz="0 0 0" rpy="0 0 0"/>
                 <geometry>
@@ -104,6 +104,6 @@
             <parent link="${parent_prefix}"/>
         </joint>
-        <link name="depth_link"></link>
-        <joint name="${frame_prefix}_to_camera_joint" type="fixed">
+        <link name="depth_link"></link> -->
+        <!-- <joint name="${frame_prefix}_to_camera_joint" type="fixed">
             <origin xyz="0 0 0" rpy="${-M_PI/2} 0 ${-M_PI/2} "/>
             <parent link="${frame_prefix}_link"/>
@@ -113,5 +113,5 @@
             <material>Gazebo/Yellow</material>
         </gazebo>
-    </xacro:macro>
+    </xacro:macro> -->
     <xacro:macro name="limo_imu" params="parent_prefix frame_prefix  *joint_pose">
         <link name='${frame_prefix}_link'>

Commit message: march 5th

File: limo_ros2/limo_description/urdf/limo_four_diff.xacro (robot description, xacro)
@@ -2,5 +2,4 @@
 <robot name="limo_four_diff" xmlns:xacro="http://ros.org/wiki/xacro">
     <xacro:include filename="$(find limo_description)/urdf/limo_xacro.xacro" />
-    <!-- <xacro:include filename="$(find limo_description)/urdf/limo_four_diff_2.gazebo" /> -->
     <!-- Variables -->
     <xacro:property name="M_PI" value="3.14159"/>
@@ -31,10 +30,4 @@
         </collision>
     </link>
-    <!-- <link name="base_footprint"/>
-    <joint name="base_joint" type="fixed">
-      <origin xyz="0 0 0.15" rpy="0 0 0"/>
-      <parent link="base_footprint"/>
-      <child link="base_link"/>
-    </joint> -->
     <link name="inertial_link">
         <inertial>
@@ -54,7 +47,4 @@
         <origin xyz="0.103 0 -0.034" rpy="0 0 0"/>
     </xacro:limo_laser>
-    <!-- <xacro:limo_depth_camera parent_prefix="base_link" frame_prefix="depth_camera">
-        <origin xyz="0.084 0 0.033" rpy="0 0 0"/>
-    </xacro:limo_depth_camera> -->
     <xacro:limo_imu parent_prefix="base_link" frame_prefix="imu">
         <origin xyz="0.0 0 -0.1" rpy="0 0 0"/>
@@ -72,207 +62,3 @@
         <origin xyz="${-wheelbase/2} ${-track/2} ${wheel_vertical_offset}" rpy="${M_PI} 0 0" />
     </xacro:limo_wheel>
-    <!-- <gazebo reference="imu_link"> -->
-    <!-- <gravity>true</gravity>
-    <sensor name="twr_imu" type="imu">
-      <always_on>true</always_on>
-      <update_rate>100</update_rate>
-      <visualize>true</visualize>
-      <imu>
-        <orientation>
-          <x>
-            <noise type="gaussian">
-              <mean>0.0</mean>
-              <stddev>2e-3</stddev>
-            </noise>
-          </x>
-          <y>
-            <noise type="gaussian">
-              <mean>0.0</mean>
-              <stddev>2e-3</stddev>
-            </noise>
-          </y>
-          <z>
-            <noise type="gaussian">
-              <mean>0.0</mean>
-              <stddev>2e-3</stddev>
-            </noise>
-          </z>
-        </orientation>
-        <angular_velocity>
-          <x>
-            <noise type="gaussian">
-              <mean>0.0</mean>
-              <stddev>2e-4</stddev>
-            </noise>
-          </x>
-          <y>
-            <noise type="gaussian">
-              <mean>0.0</mean>
-              <stddev>2e-4</stddev>
-            </noise>
-          </y>
-          <z>
-            <noise type="gaussian">
-              <mean>0.0</mean>
-              <stddev>2e-4</stddev>
-            </noise>
-          </z>
-        </angular_velocity>
-        <linear_acceleration>
-          <x>
-            <noise type="gaussian">
-              <mean>0.0</mean>
-              <stddev>1.7e-2</stddev>
-            </noise>
-          </x>
-          <y>
-            <noise type="gaussian">
-              <mean>0.0</mean>
-              <stddev>1.7e-2</stddev>
-            </noise>
-          </y>
-          <z>
-            <noise type="gaussian">
-              <mean>0.0</mean>
-              <stddev>1.7e-2</stddev>
-            </noise>
-          </z>
-        </linear_acceleration>
-      </imu>
-      <plugin name="two_wheeled_robot_imu" filename="libgazebo_ros_imu_sensor.so">
-        <initial_orientation_as_reference>false</initial_orientation_as_reference>
-        <frame_name>imu_link</frame_name>
-        <ros>
-          <namespace>/imu</namespace>
-          <remapping>~/out:=data</remapping>
-        </ros>
-      </plugin>
-    </sensor>
-</gazebo> -->
-<!-- <gazebo reference="laser_link">
-    <sensor name="laser" type="ray">
-      <always_on>true</always_on>
-      <visualize>true</visualize>
-      <update_rate>10</update_rate>
-      <ray>
-        <scan>
-          <horizontal>
-            <samples>120</samples>
-            <resolution>1.000000</resolution>
-            <min_angle>-3.14159</min_angle>
-            <max_angle>3.14159</max_angle>
-          </horizontal>
-        </scan>
-        <range>
-          <min>0.3</min>
-          <max>15.0</max>
-          <resolution>0.015</resolution>
-        </range>
-        <noise>
-          <type>gaussian</type>
-          <mean>0.0</mean>
-          <stddev>0.01</stddev>
-        </noise>
-      </ray>
-      <plugin name="scan" filename="libgazebo_ros_ray_sensor.so">
-        <ros>
-          <remapping>~/out:=scan</remapping>
-        </ros>
-        <output_type>sensor_msgs/LaserScan</output_type>
-        <frame_name>laser_link</frame_name>
-      </plugin>
-    </sensor>
-  </gazebo> -->
-    <!-- <gazebo reference="front_left_wheel">
-        <mu1>100</mu1>
-        <mu2>100</mu2>
-        <kp>10000000.0</kp>
-        <kd>1.0</kd>
-        <minDepth>0.01</minDepth>
-        <fdir1>1 0 0</fdir1>
-        <maxContacts value="64"/>
-    </gazebo>
-    <gazebo reference="front_right_wheel">
-        <mu1>100</mu1>
-        <mu2>100</mu2>
-        <kp>10000000.0</kp>
-        <kd>1.0</kd>
-        <minDepth>0.01</minDepth>
-        <fdir1>1 0 0</fdir1>
-        <maxContacts value="64"/>
-    </gazebo>
-    <gazebo reference="rear_left_wheel">
-        <mu1>100</mu1>
-        <mu2>100</mu2>
-        <kp>10000000.0</kp>
-        <kd>1.0</kd>
-        <minDepth>0.01</minDepth>
-        <fdir1>1 0 0</fdir1>
-        <maxContacts value="64"/>
-    </gazebo>
-    <gazebo reference="rear_right_wheel">
-        <mu1>100</mu1>
-        <mu2>100</mu2>
-        <kp>10000000.0</kp>
-        <kd>1.0</kd>
-        <minDepth>0.01</minDepth>
-        <fdir1>1 0 0</fdir1>
-        <maxContacts value="64"/>
-    </gazebo>
-    <gazebo>
-        <plugin name="four_diff_controller" filename="libgazebo_ros_diff_drive.so">
-        <update_rate>50</update_rate>
-        <num_wheel_pairs>2</num_wheel_pairs>
-        <left_joint>front_left_wheel</left_joint>
-        <right_joint>front_right_wheel</right_joint>
-        <left_joint>rear_left_wheel</left_joint>
-        <right_joint>rear_right_wheel</right_joint>
-        <wheel_separation>0.172</wheel_separation>
-        <wheel_diameter>0.09</wheel_diameter>
-        <max_wheel_torque>20</max_wheel_torque>
-        <max_wheel_acceleration>1.0</max_wheel_acceleration>
-        <command_topic>cmd_vel</command_topic>
-        <publish_odom>true</publish_odom>
-        <publish_odom_tf>true</publish_odom_tf>
-        <publish_wheel_tf>true</publish_wheel_tf>
-        <odometry_topic>odom</odometry_topic>
-        <odometry_frame>odom</odometry_frame>
-        <robot_base_frame>base_footprint</robot_base_frame>
-        <odometry_source>1</odometry_source>
-        <ros>
-            <remapping>odom:=/odometry</remapping>
-        </ros>
-        </plugin>
-    </gazebo> -->
-        <!-- <gazebo reference="depth_camera_link">
-          <sensor name="sensor_camera" type="depth">
-            <pose>0.0 0.0 0.0 0.0 0.0 0.0</pose>
-            <always_on>0</always_on>
-            <update_rate>1</update_rate>
-            <camera name="limo_camera">
-              <distortion>
-                <k1>0.1</k1>
-                <k2>0.2</k2>
-                <k3>0.3</k3>
-                <p1>0.4</p1>
-                <p2>0.5</p2>
-                <center>0.5 0.5</center>
-              </distortion>
-            </camera>
-            <plugin name="gazebo_ros_depth_camera_sensor" filename="libgazebo_ros_camera.so">
-              <ros>
-                <namespace>/limo</namespace>
-                <argument>limo_camera/image_raw:=limo_camera/image</argument>
-                <argument>limo_camera/image_depth:=limo_camera/depth/camera_image_depth</argument>
-                <argument>limo_camera/camera_info:=limo_camera/camera_info_raw</argument>
-                <argument>limo_camera/camera_info_depth:=limo_camera/camera_info_depth</argument>
-                <argument>limo_camera/points:=limo_camera/camera_points</argument>
-              </ros>
-              <camera_name>depth_camera_link</camera_name>
-              <frame_name>depth_camera_link</frame_name>
-              <hack_baseline>0.07</hack_baseline>
-              <min_depth>0.001</min_depth>
-            </plugin>
-        </sensor>
-          </gazebo> -->
 </robot>

File: limo_ros2/limo_description/urdf/limo_xacro.xacro (robot description, xacro)
@@ -68,50 +68,4 @@
         </gazebo>
     </xacro:macro>
-    <!-- <xacro:macro name="limo_depth_camera" params="parent_prefix frame_prefix *joint_pose">
-        <link name='${frame_prefix}_link'>
-            <pose>0 0 0 0 0 0</pose>
-            <inertial>
-                <mass value="0.1"/>
-                <origin xyz="0.0 0 0" rpy="0 0 0"/>
-                <inertia
-                    ixx="1e-6" ixy="0" ixz="0"
-                    iyy="1e-6" iyz="0"
-                    izz="1e-6"
-                />
-            </inertial> -->
-            <!-- <visual name='depth_camera_visual'>
-                <origin xyz="0 0 0" rpy="0 0 0"/>
-                <geometry>
-                    <box size="0.02 0.06 0.015"/>
-                </geometry>
-                <material name='depth_camera_material'>
-                    <ambient>0.1 0.1 0.1 1</ambient>
-                    <diffuse>0.1 0.1 0.2 1</diffuse>
-                    <specular>0 0 0 0</specular>
-                    <emissive>0 0 0 1</emissive>
-                </material>
-            </visual> -->
-            <!-- <collision name='depth_camera_collision'>
-                <origin xyz="0 0 0" rpy="0 0 0"/>
-                <geometry>
-                    <box size="0.02 0.06 0.015"/>
-                </geometry>
-            </collision>
-        </link>
-        <joint type="fixed" name="depth_camera_joint">
-            <xacro:insert_block name="joint_pose"/>
-            <child link="${frame_prefix}_link"/>
-            <parent link="${parent_prefix}"/>
-        </joint>
-        <link name="depth_link"></link> -->
-        <!-- <joint name="${frame_prefix}_to_camera_joint" type="fixed">
-            <origin xyz="0 0 0" rpy="${-M_PI/2} 0 ${-M_PI/2} "/>
-            <parent link="${frame_prefix}_link"/>
-            <child link="depth_link"/>
-          </joint>
-        <gazebo reference="${frame_prefix}_link">
-            <material>Gazebo/Yellow</material>
-        </gazebo>
-    </xacro:macro> -->
     <xacro:macro name="limo_imu" params="parent_prefix frame_prefix  *joint_pose">
         <link name='${frame_prefix}_link'>
